File: switch_main_v5/2v5_buck_converter.kicad_sch (KiCad schematic)
At the start: 12 parts, among them U1304 TPS62290TDRVRQ1

Commit message: Updated 1v0_buck_converter feedback resistors
Parts:
- renumbered C1330 to C3701, C1331 to C3702, C1332 to C3703, C1333 to C3704, C1334 to C3705, C1335 to C3706, C1336 to C3707, L1303 to L3701, R1311 to R3701, R1312 to R3702, TP1304 to TP3701, U1304 to U3701
Changed lines of the file:
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@@
 		(dnp no)
 		(fields_autoplaced yes)
-		(property "Reference" "#PWR01329"
+		(property "Reference" "#PWR03701"
 			(at 73.66 113.03 0)
 			(effects
@@
 			(project "switch_main_v5"
 				(path "/a5e57332-4284-4d3c-ab3c-13bc0ddb29b6/b1ff42f5-7cae-489e-9f8e-588cc93f3151/d017dddd-15df-4565-b589-89c8c78bc85c/9430147e-67d1-4fa5-a888-19b664a1bd8a"
-					(reference "#PWR01329")
+					(reference "#PWR03701")
 					(unit 1)
 				)
@@
 		(on_board yes)
 		(dnp no)
-		(property "Reference" "C1330"
+		(property "Reference" "C3701"
 			(at 76.2 97.7962 0)
 			(effects
@@
 			(project "switch_main_v5"
 				(path "/a5e57332-4284-4d3c-ab3c-13bc0ddb29b6/b1ff42f5-7cae-489e-9f8e-588cc93f3151/d017dddd-15df-4565-b589-89c8c78bc85c/9430147e-67d1-4fa5-a888-19b664a1bd8a"
-					(reference "C1330")
+					(reference "C3701")
 					(unit 1)
 				)
@@
 		(dnp no)
 		(fields_autoplaced yes)
-		(property "Reference" "L1303"
+		(property "Reference" "L3701"
 			(at 162.56 85.09 0)
 			(effects
@@
 			(project "switch_main_v5"
 				(path "/a5e57332-4284-4d3c-ab3c-13bc0ddb29b6/b1ff42f5-7cae-489e-9f8e-588cc93f3151/d017dddd-15df-4565-b589-89c8c78bc85c/9430147e-67d1-4fa5-a888-19b664a1bd8a"
-					(reference "L1303")
+					(reference "L3701")
 					(unit 1)
 				)
@@
 		(dnp no)
 		(fields_autoplaced yes)
-		(property "Reference" "C1335"
+		(property "Reference" "C3706"
 			(at 213.36 97.7962 0)
 			(effects
@@
 			(project "switch_main_v5"
 				(path "/a5e57332-4284-4d3c-ab3c-13bc0ddb29b6/b1ff42f5-7cae-489e-9f8e-588cc93f3151/d017dddd-15df-4565-b589-89c8c78bc85c/9430147e-67d1-4fa5-a888-19b664a1bd8a"
-					(reference "C1335")
+					(reference "C3706")
 					(unit 1)
 				)
@@
 		(dnp no)
 		(fields_autoplaced yes)
-		(property "Reference" "R1311"
+		(property "Reference" "R3701"
 			(at 175.26 97.7899 0)
 			(effects
@@
 			(project "switch_main_v5"
 				(path "/a5e57332-4284-4d3c-ab3c-13bc0ddb29b6/b1ff42f5-7cae-489e-9f8e-588cc93f3151/d017dddd-15df-4565-b589-89c8c78bc85c/9430147e-67d1-4fa5-a888-19b664a1bd8a"
-					(reference "R1311")
+					(reference "R3701")
 					(unit 1)
 				)
@@
 		(dnp no)
 		(fields_autoplaced yes)
-		(property "Reference" "#PWR01332"
+		(property "Reference" "#PWR03704"
 			(at 172.72 123.19 0)
 			(effects
@@
 			(project "switch_main_v5"
 				(path "/a5e57332-4284-4d3c-ab3c-13bc0ddb29b6/b1ff42f5-7cae-489e-9f8e-588cc93f3151/d017dddd-15df-4565-b589-89c8c78bc85c/9430147e-67d1-4fa5-a888-19b664a1bd8a"
-					(reference "#PWR01332")
+					(reference "#PWR03704")
 					(unit 1)
 				)
@@
 		(dnp no)
 		(fields_autoplaced yes)
-		(property "Reference" "C1334"
+		(property "Reference" "C3705"
 			(at 200.66 97.7962 0)
 			(effects
@@
 			(project "switch_main_v5"
 				(path "/a5e57332-4284-4d3c-ab3c-13bc0ddb29b6/b1ff42f5-7cae-489e-9f8e-588cc93f3151/d017dddd-15df-4565-b589-89c8c78bc85c/9430147e-67d1-4fa5-a888-19b664a1bd8a"
-					(reference "C1334")
+					(reference "C3705")
 					(unit 1)
 				)
@@
 		(on_board yes)
 		(dnp no)
-		(property "Reference" "C1331"
+		(property "Reference" "C3702"
 			(at 88.9 97.7962 0)
 			(effects
@@
 			(project "switch_main_v5"
 				(path "/a5e57332-4284-4d3c-ab3c-13bc0ddb29b6/b1ff42f5-7cae-489e-9f8e-588cc93f3151/d017dddd-15df-4565-b589-89c8c78bc85c/9430147e-67d1-4fa5-a888-19b664a1bd8a"
-					(reference "C1331")
+					(reference "C3702")
 					(unit 1)
 				)
@@
 		(dnp no)
 		(fields_autoplaced yes)
-		(property "Reference" "#PWR01330"
+		(property "Reference" "#PWR03702"
 			(at 111.76 123.19 0)
 			(effects
@@
 			(project "switch_main_v5"
 				(path "/a5e57332-4284-4d3c-ab3c-13bc0ddb29b6/b1ff42f5-7cae-489e-9f8e-588cc93f3151/d017dddd-15df-4565-b589-89c8c78bc85c/9430147e-67d1-4fa5-a888-19b664a1bd8a"
-					(reference "#PWR01330")
+					(reference "#PWR03702")
 					(unit 1)
 				)
@@
 		(on_board yes)
 		(dnp no)
-		(property "Reference" "C1333"
+		(property "Reference" "C3704"
 			(at 187.96 97.7962 0)
 			(effects
@@
 			(project "switch_main_v5"
 				(path "/a5e57332-4284-4d3c-ab3c-13bc0ddb29b6/b1ff42f5-7cae-489e-9f8e-588cc93f3151/d017dddd-15df-4565-b589-89c8c78bc85c/9430147e-67d1-4fa5-a888-19b664a1bd8a"
-					(reference "C1333")
+					(reference "C3704")
 					(unit 1)
 				)
@@
 		(on_board yes)
 		(dnp no)
-		(property "Reference" "TP1304"
+		(property "Reference" "TP3701"
 			(at 233.68 88.9 0)
 			(effects
@@
 			(project "switch_main_v5"
 				(path "/a5e57332-4284-4d3c-ab3c-13bc0ddb29b6/b1ff42f5-7cae-489e-9f8e-588cc93f3151/d017dddd-15df-4565-b589-89c8c78bc85c/9430147e-67d1-4fa5-a888-19b664a1bd8a"
-					(reference "TP1304")
+					(reference "TP3701")
 					(unit 1)
 				)
@@
 		(dnp no)
 		(fields_autoplaced yes)
-		(property "Reference" "#PWR01331"
+		(property "Reference" "#PWR03703"
 			(at 147.32 123.19 0)
 			(effects
@@
 			(project "switch_main_v5"
 				(path "/a5e57332-4284-4d3c-ab3c-13bc0ddb29b6/b1ff42f5-7cae-489e-9f8e-588cc93f3151/d017dddd-15df-4565-b589-89c8c78bc85c/9430147e-67d1-4fa5-a888-19b664a1bd8a"
-					(reference "#PWR01331")
+					(reference "#PWR03703")
 					(unit 1)
 				)
@@
 		(dnp no)
 		(fields_autoplaced yes)
-		(property "Reference" "U1304"
+		(property "Reference" "U3701"
 			(at 129.54 86.36 0)
 			(effects
@@
 			(project "switch_main_v5"
 				(path "/a5e57332-4284-4d3c-ab3c-13bc0ddb29b6/b1ff42f5-7cae-489e-9f8e-588cc93f3151/d017dddd-15df-4565-b589-89c8c78bc85c/9430147e-67d1-4fa5-a888-19b664a1bd8a"
-					(reference "U1304")
+					(reference "U3701")
 					(unit 1)
 				)
@@
 		(dnp no)
 		(fields_autoplaced yes)
-		(property "Reference" "R1312"
+		(property "Reference" "R3702"
 			(at 175.26 110.4899 0)
 			(effects
@@
 			(project "switch_main_v5"
 				(path "/a5e57332-4284-4d3c-ab3c-13bc0ddb29b6/b1ff42f5-7cae-489e-9f8e-588cc93f3151/d017dddd-15df-4565-b589-89c8c78bc85c/9430147e-67d1-4fa5-a888-19b664a1bd8a"
-					(reference "R1312")
+					(reference "R3702")
 					(unit 1)
 				)
@@
 		(dnp no)
 		(fields_autoplaced yes)
-		(property "Reference" "C1336"
+		(property "Reference" "C3707"
 			(at 226.06 97.7962 0)
 			(effects
@@
 			(project "switch_main_v5"
 				(path "/a5e57332-4284-4d3c-ab3c-13bc0ddb29b6/b1ff42f5-7cae-489e-9f8e-588cc93f3151/d017dddd-15df-4565-b589-89c8c78bc85c/9430147e-67d1-4fa5-a888-19b664a1bd8a"
-					(reference "C1336")
+					(reference "C3707")
 					(unit 1)
 				)
@@
 		(on_board yes)
 		(dnp no)
-		(property "Reference" "C1332"
+		(property "Reference" "C3703"
 			(at 101.6 97.7962 0)
 			(effects
@@
 			(project "switch_main_v5"
 				(path "/a5e57332-4284-4d3c-ab3c-13bc0ddb29b6/b1ff42f5-7cae-489e-9f8e-588cc93f3151/d017dddd-15df-4565-b589-89c8c78bc85c/9430147e-67d1-4fa5-a888-19b664a1bd8a"
-					(reference "C1332")
+					(reference "C3703")
 					(unit 1)
 				)
@@
 		(dnp no)
 		(fields_autoplaced yes)
-		(property "Reference" "#PWR01333"
+		(property "Reference" "#PWR03705"
 			(at 223.52 113.03 0)
 			(effects
@@
 			(project "switch_main_v5"
 				(path "/a5e57332-4284-4d3c-ab3c-13bc0ddb29b6/b1ff42f5-7cae-489e-9f8e-588cc93f3151/d017dddd-15df-4565-b589-89c8c78bc85c/9430147e-67d1-4fa5-a888-19b664a1bd8a"
-					(reference "#PWR01333")
-					(unit 1)
-				)
+					(reference "#PWR03705")
+					(unit 1)
+				)
