File: switch_main_v5/1000base-t1-cdn-shield.kicad_sch (KiCad schematic)
At the start: 9 parts, among them T3301 74930100

Commit message: Changed main 3V3 regulator to 3A, added switch 2 crystal & other changes
Parts:
- renumbered C3301 to C1801, C3302 to C1802, C3303 to C1803, D3301 to D1801, D3302 to D1802, D3303 to D1803, FL3301 to FL1801, R3301 to R1801, T3301 to T1801
Connections:
- net SHIELD renamed SHIELD0

Commit message: Tidied schematic and PCB
Parts:
- removed C1801: 100n, Capacitor_SMD:C_0402_1005Metric, symbol Device:C_Small
- removed C1802: 100n, Capacitor_SMD:C_0603_1608Metric, symbol Device:C_Small
- removed C1803: 1n, Capacitor_SMD:C_0805_2012Metric, symbol Device:C_Small
- removed D1801: 824012823, project_footprints:824012823, symbol TVS:824012823
- removed D1802, D1803: SZESD7241N2T5G, project_footprints:SZESD7462N2T5G, symbol TVS:SZESD7241N2T5G
- removed FL1801: ACT1210G-800-2P-TL10, project_footprints:ACT1210G, symbol COMM-CMC:ACT1210G-800-2P-TL10
- removed R1801: 100R, Resistor_SMD:R_0402_1005Metric, symbol Device:R_Small
- removed T1801: 74930100, project_footprints:74930100, symbol COMM-TRANSFORMER:74930100
- added C3301: 100n, Capacitor_SMD:C_0603_1608Metric, symbol Device:C_Small
- added C3302: 100n, Capacitor_SMD:C_0402_1005Metric, symbol Device:C_Small
- added C3303: 1n, Capacitor_SMD:C_0805_2012Metric, symbol Device:C_Small
- added D3301, D3303: SZESD7241N2T5G, project_footprints:SZESD7462N2T5G, symbol TVS:SZESD7241N2T5G
- added D3302: 824012823, project_footprints:824012823, symbol TVS:824012823
- added FL3301: ACT1210G-800-2P-TL10, project_footprints:ACT1210G, symbol COMM-CMC:ACT1210G-800-2P-TL10
- added R3301: 100R, Resistor_SMD:R_0402_1005Metric, symbol Device:R_Small
- added T3301: 74930100, project_footprints:74930100, symbol COMM-TRANSFORMER:74930100
Connections:
- net CTP: now also C3302.1, T3301.5 (PM)
- net CTS1: now also C3301.2, T3301.4 (OUT1B)
- net CTS2: now also C3301.1, R3301.2, T3301.3 (OUT2A)
- net GND1: now also C3302.2, D3302.3, D3302.4
- net MDI_IN.TRXN: now also D3302.1, D3302.6, FL3301.3
- net MDI_IN.TRXP: now also D3302.2, D3302.5, FL3301.4
- net MDI_OUT.TRXN: now also D3303.2 (A2), T3301.7 (OUT2B)
- net MDI_OUT.TRXP: now also D3301.2 (A2), T3301.6 (OUT1A)
- net SHIELD0: now also C3303.2, D3301.1 (A1), D3303.1 (A1)
- net TERM: now also C3303.1, R3301.1
- net TRXN: now also FL3301.2, T3301.2 (IN-)
- net TRXP: now also FL3301.1, T3301.1 (IN+)
