File: switch_main_v5/1000base-t1-phy.kicad_sch (KiCad schematic)
At the start: 37 parts, among them Q1301 DMN21D2UFB-7B, Q1302 DMP21D0UFB-7B, U1301 TPS62290TDRVRQ1, U1302 88Q2112-A2-NYD2A000-P123

Commit message: Changed main 3V3 regulator to 3A, added switch 2 crystal & other changes
Parts:
- removed C1301, C1302, C1304, C1306, C1307: 4u7, Capacitor_SMD:C_0402_1005Metric, symbol Device:C_Small
- removed C1303: 22p, Capacitor_SMD:C_0402_1005Metric, symbol Device:C_Small
- removed L1301: 78438313015, project_footprints:L_Wurth_WE-MAIA-1610, symbol PWR-IND:1610_78438313015
- removed R1304: 180k, Resistor_SMD:R_0402_1005Metric, symbol Device:R_Small
- removed R1305: 360k, Resistor_SMD:R_0402_1005Metric, symbol Device:R_Small
- removed TP1302: 1.5mm, TestPoint:TestPoint_Pad_D1.5mm, symbol Connector:TestPoint_Small
- removed U1301: TPS62290TDRVRQ1, project_footprints:SON65P200X200X80-7N, symbol PWR-SMPS:TPS62290TDRVRQ1
Connections:
- net +1V8 renamed +1V8_PHY
Other:
- moved on the sheet: C1305, C1308, C1309, C1310, C1311, C1312, C1313, C1314, C1315, C1316, C1317, C1318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

Commit message: PHY3 RGMII routed and length matched
Changed lines of the file:
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@@
+	)
+	(junction
+		(at 226.06 78.74)
+		(diameter 0)
+		(color 0 0 0 0)
 	)
 	(junction
@@
 		)
 	)
+	(wire
+		(pts
+			(xy 223.52 78.74) (xy 226.06 78.74)
+		)
+		(stroke
+			(width 0)
+			(type default)
+		)
+	)
 	(bus
 		(pts
@@
 			(width 0)
 			(type default)
-		)
-	)
-	(label "0V9"
-		(at 226.06 78.74 0)
-		(effects
-			(font
-				(size 1.27 1.27)
-			)
-			(justify left bottom)
 		)
 	)
@@
 		)
 	)
+	(hierarchical_label "0V9"
+		(shape input)
+		(at 223.52 78.74 180)
+		(effects
+			(font
+				(size 1.27 1.27)
+			)
+			(justify right)
+		)
+	)

Commit message: Tidied schematic and PCB
Parts:
- renumbered C1308 to C2001, C1310 to C2002, C1313 to C2003, C1315 to C2004, C1317 to C2005, C1319 to C2006, C1321 to C2007, C1309 to C2008, C1311 to C2009, C1312 to C2010, C1316 to C2011, C1318 to C2012, C1320 to C2013, C1322 to C2014, C1314 to C2015, C1305 to C2016, Q1302 to Q2001, Q1301 to Q2002, R1302 to R2001, R1308 to R2002, R1307 to R2003, R1301 to R2004, R1306 to R2005, R1303 to R2006, TP1301 to TP2001, U1302 to U2001
