File: switch_main_v5/10base-t1s-phy.kicad_sch (KiCad schematic)
At the start: 20 parts, among them U1601 LAN8671C2-E_U3B

Commit message: Tidied schematic and PCB
Parts:
- renumbered C1601 to C2501, C1604 to C2502, C1607 to C2503, C1610 to C2504, C1611 to C2505, C1602 to C2506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
