File: switch_main_v5/1v0_buck_converter.kicad_sch (KiCad schematic)
At the start: 12 parts, among them U3801 TPS62290TDRVRQ1

Commit message: Updated 1v0_buck_converter feedback resistors
Parts:
- removed C3801, C3802, C3803, C3805, C3806, C3807: 4u7, Capacitor_SMD:C_0402_1005Metric, symbol Device:C_Small
- removed C3804: 22p, Capacitor_SMD:C_0402_1005Metric, symbol Device:C_Small
- removed L3801: 78438313015, project_footprints:L_Wurth_WE-MAIA-1610, symbol PWR-IND:1610_78438313015
- removed R3801, R3802: 180k, Resistor_SMD:R_0402_1005Metric, symbol Device:R_Small
- removed TP3801: 1.5mm, TestPoint:TestPoint_Pad_D1.5mm, symbol Connector:TestPoint_Small
- removed U3801: TPS62290TDRVRQ1, project_footprints:SON65P200X200X80-7N, symbol PWR-SMPS:TPS62290TDRVRQ1
- added C3901, C3902, C3903, C3905, C3906, C3907: 4u7, Capacitor_SMD:C_0402_1005Metric, symbol Device:C_Small
- added C3904: 22p, Capacitor_SMD:C_0402_1005Metric, symbol Device:C_Small
- added L3901: 78438313015, project_footprints:L_Wurth_WE-MAIA-1610, symbol PWR-IND:1610_78438313015
- added R3901: 120k, Resistor_SMD:R_0402_1005Metric, symbol Device:R_Small
- added R3902: 180k, Resistor_SMD:R_0402_1005Metric, symbol Device:R_Small
- added TP3901: 1.5mm, TestPoint:TestPoint_Pad_D1.5mm, symbol Connector:TestPoint_Small
- added U3901: TPS62290TDRVRQ1, project_footprints:SON65P200X200X80-7N, symbol PWR-SMPS:TPS62290TDRVRQ1
Connections:
- net FB_1V2: now also C3904.2, R3901.2, R3902.1, U3901.3 (FB)
- net GND1: now also C3901.2, C3902.2, C3903.2, C3905.2, C3906.2, C3907.2, R3902.2, U3901.2 (MODE), U3901.6 (GND), U3901.7 (EP)
- net SW_1V2: now also L3901.1, U3901.1 (SW)
- net VIN: now also C3901.1, C3902.1, C3903.1, U3901.4 (EN), U3901.5 (VIN)
- net VOUT: now also C3904.1, C3905.1, C3906.1, C3907.1, L3901.2, R3901.1, TP3901.1

Commit message: 1V0 Rail done
Parts:
- removed C3903: 4u7, Capacitor_SMD:C_0402_1005Metric, symbol Device:C_Small
Connections:
- net FB_1V2 renamed FB
- net SW_1V2 renamed SW
Other:
- moved on the sheet: C3901, C3902

Commit message: Placed most remaining passives and test points
Connections:
- net GND1: no longer U3901.2 (MODE)
- net VOUT: now also U3901.2 (MODE)
Changed lines of the file:
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@@
+		)
+	)
+	(text_box "MODE >=1.0V means FPWM mode (necessary for PHY ripple specs)"
+		(exclude_from_sim no)
+		(at 83.82 114.3 0)
+		(size 25.4 7.62)
+		(margins 0.9525 0.9525 0.9525 0.9525)
+		(stroke
+			(width 0)
+			(type solid)
+		)
+		(fill
+			(type none)
+		)
+		(effects
+			(font
+				(size 1.27 1.27)
+			)
+			(justify left top)
 		)
 	)
@@
 	)
 	(junction
-		(at 116.84 111.76)
-		(diameter 0)
-		(color 0 0 0 0)
-	)
-	(junction
 		(at 228.6 91.44)
 		(diameter 0)
@@
 	(wire
 		(pts
-			(xy 119.38 106.68) (xy 116.84 106.68)
-		)
-		(stroke
-			(width 0)
-			(type default)
-		)
-	)
-	(wire
-		(pts
 			(xy 116.84 91.44) (xy 119.38 91.44)
 		)
@@
 	(wire
 		(pts
-			(xy 116.84 106.68) (xy 116.84 111.76)
-		)
-		(stroke
-			(width 0)
-			(type default)
-		)
-	)
-	(wire
-		(pts
 			(xy 203.2 91.44) (xy 203.2 93.98)
 		)
@@
 		(pts
 			(xy 203.2 99.06) (xy 203.2 101.6)
+		)
+		(stroke
+			(width 0)
+			(type default)
+		)
+	)
+	(wire
+		(pts
+			(xy 111.76 106.68) (xy 119.38 106.68)
 		)
 		(stroke
@@
 		(effects
 			(font
+				(size 1.27 1.27)
+			)
+			(justify left bottom)
+		)
+	)
+	(label "VOUT"
+		(at 111.76 106.68 0)
+		(effects
+			(font

Commit message: Tidied schematic and PCB
Parts:
- renumbered C3901 to C901, C3902 to C902, C3904 to C903, C3905 to C904, C3906 to C905, C3907 to C906, L3901 to L901, R3901 to R901, R3902 to R902, TP3901 to TP901, U3901 to U901
Connections:
- net VIN: now also U901.2 (MODE)
- net VOUT: no longer U901.2 (MODE)
Other:
- moved on the sheet: C901, C902, C903, C904, C905, C906, L901, R901, R902, TP901, U901
