File: switch_main_v5/1v8_buck_converter.kicad_sch (KiCad schematic)
At the start: 12 parts, among them U3401 TPS62290TDRVRQ1

Commit message: Updated 1v0_buck_converter feedback resistors
Parts:
- removed C3401, C3402, C3403, C3405, C3406, C3407: 4u7, Capacitor_SMD:C_0402_1005Metric, symbol Device:C_Small
- removed C3404: 22p, Capacitor_SMD:C_0402_1005Metric, symbol Device:C_Small
- removed L3401: 78438313015, project_footprints:L_Wurth_WE-MAIA-1610, symbol PWR-IND:1610_78438313015
- removed R3401: 360k, Resistor_SMD:R_0402_1005Metric, symbol Device:R_Small
- removed R3402: 180k, Resistor_SMD:R_0402_1005Metric, symbol Device:R_Small
- removed TP3401: 1.5mm, TestPoint:TestPoint_Pad_D1.5mm, symbol Connector:TestPoint_Small
- removed U3401: TPS62290TDRVRQ1, project_footprints:SON65P200X200X80-7N, symbol PWR-SMPS:TPS62290TDRVRQ1
- added C1201, C1202, C1203, C1205, C1206, C1207: 4u7, Capacitor_SMD:C_0402_1005Metric, symbol Device:C_Small
- added C1204: 22p, Capacitor_SMD:C_0402_1005Metric, symbol Device:C_Small
- added L1201: 78438313015, project_footprints:L_Wurth_WE-MAIA-1610, symbol PWR-IND:1610_78438313015
- added R1201: 360k, Resistor_SMD:R_0402_1005Metric, symbol Device:R_Small
- added R1202: 180k, Resistor_SMD:R_0402_1005Metric, symbol Device:R_Small
- added TP1201: 1.5mm, TestPoint:TestPoint_Pad_D1.5mm, symbol Connector:TestPoint_Small
- added U1201: TPS62290TDRVRQ1, project_footprints:SON65P200X200X80-7N, symbol PWR-SMPS:TPS62290TDRVRQ1
Connections:
- net FB_1V8: now also C1204.2, R1201.2, R1202.1, U1201.3 (FB)
- net GND1: now also C1201.2, C1202.2, C1203.2, C1205.2, C1206.2, C1207.2, R1202.2, U1201.2 (MODE), U1201.6 (GND), U1201.7 (EP)
- net SW_1V8: now also L1201.1, U1201.1 (SW)
- net VIN: now also C1201.1, C1202.1, C1203.1, U1201.4 (EN), U1201.5 (VIN)
- net VOUT: now also C1204.1, C1205.1, C1206.1, C1207.1, L1201.2, R1201.1, TP1201.1

Commit message: Moved 0V9 regulators
Parts:
- removed C1201: 4u7, Capacitor_SMD:C_0402_1005Metric, symbol Device:C_Small
Changed lines of the file:
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@@
-	)
-	(junction
-		(at 73.66 93.98)
-		(diameter 0)
-		(color 0 0 0 0)
 	)
 	(junction
@@
 	)
 	(junction
-		(at 73.66 104.14)
-		(diameter 0)
-		(color 0 0 0 0)
-	)
-	(junction
 		(at 210.82 93.98)
 		(diameter 0)
@@
 	(wire
 		(pts
-			(xy 73.66 104.14) (xy 86.36 104.14)
-		)
-		(stroke
-			(width 0)
-			(type default)
-		)
-	)
-	(wire
-		(pts
 			(xy 223.52 104.14) (xy 210.82 104.14)
 		)
@@
 	(wire
 		(pts
-			(xy 73.66 93.98) (xy 86.36 93.98)
-		)
-		(stroke
-			(width 0)
-			(type default)
-		)
-	)
-	(wire
-		(pts
-			(xy 71.12 93.98) (xy 73.66 93.98)
+			(xy 83.82 93.98) (xy 86.36 93.98)
 		)
 		(stroke
@@
 	(wire
 		(pts
-			(xy 73.66 106.68) (xy 73.66 104.14)
+			(xy 86.36 106.68) (xy 86.36 104.14)
 		)
 		(stroke
@@
 	(wire
 		(pts
+			(xy 185.42 93.98) (xy 185.42 96.52)
+		)
+		(stroke
+			(width 0)
+			(type default)
+		)
+	)
+	(wire
+		(pts
+			(xy 198.12 101.6) (xy 198.12 104.14)
+		)
+		(stroke
+			(width 0)
+			(type default)
+		)
+	)
+	(wire
+		(pts
+			(xy 99.06 101.6) (xy 99.06 104.14)
+		)
+		(stroke
+			(width 0)
+			(type default)
+		)
+	)
+	(wire
+		(pts
+			(xy 223.52 93.98) (xy 223.52 96.52)
+		)
+		(stroke
+			(width 0)
+			(type default)
+		)
+	)
+	(wire
+		(pts
+			(xy 210.82 93.98) (xy 210.82 96.52)
+		)
+		(stroke
+			(width 0)
+			(type default)
+		)
+	)
+	(wire
+		(pts
+			(xy 185.42 106.68) (xy 172.72 106.68)
+		)
+		(stroke
+			(width 0)
+			(type default)
+		)
+	)
+	(wire
+		(pts
+			(xy 172.72 93.98) (xy 185.42 93.98)
+		)
+		(stroke
+			(width 0)
+			(type default)
+		)
+	)
+	(wire
+		(pts
+			(xy 86.36 93.98) (xy 99.06 93.98)
+		)
+		(stroke
+			(width 0)
+			(type default)
+		)
+	)
+	(wire
+		(pts
+			(xy 144.78 93.98) (xy 157.48 93.98)
+		)
+		(stroke
+			(width 0)
+			(type default)
+		)
+	)
+	(wire
+		(pts
+			(xy 198.12 93.98) (xy 210.82 93.98)
+		)
+		(stroke
+			(width 0)
+			(type default)
+		)
+	)
+	(wire
+		(pts
+			(xy 114.3 109.22) (xy 111.76 109.22)
+		)
+		(stroke
+			(width 0)
+			(type default)
+		)
+	)
+	(wire
+		(pts
+			(xy 198.12 93.98) (xy 198.12 96.52)
+		)
+		(stroke
+			(width 0)
+			(type default)
+		)
+	)
+	(wire
+		(pts
+			(xy 144.78 104.14) (xy 172.72 104.14)
+		)
+		(stroke
+			(width 0)
+			(type default)
+		)
+	)
+	(wire
+		(pts
+			(xy 172.72 106.68) (xy 172.72 109.22)
+		)
+		(stroke
+			(width 0)
+			(type default)
+		)
+	)
+	(wire
+		(pts
 			(xy 86.36 93.98) (xy 86.36 96.52)
-		)
-		(stroke
-			(width 0)
-			(type default)
-		)
-	)
-	(wire
-		(pts
-			(xy 185.42 93.98) (xy 185.42 96.52)
-		)
-		(stroke
-			(width 0)
-			(type default)
-		)
-	)
-	(wire
-		(pts
-			(xy 198.12 101.6) (xy 198.12 104.14)
-		)
-		(stroke
-			(width 0)
-			(type default)
-		)
-	)
-	(wire
-		(pts
-			(xy 99.06 101.6) (xy 99.06 104.14)
-		)
-		(stroke
-			(width 0)
-			(type default)
-		)
-	)
-	(wire
-		(pts
-			(xy 223.52 93.98) (xy 223.52 96.52)
-		)
-		(stroke
-			(width 0)
-			(type default)
-		)
-	)
-	(wire
-		(pts
-			(xy 210.82 93.98) (xy 210.82 96.52)
-		)
-		(stroke
-			(width 0)
-			(type default)
-		)
-	)
-	(wire
-		(pts
-			(xy 185.42 106.68) (xy 172.72 106.68)
-		)
-		(stroke
-			(width 0)
-			(type default)
-		)
-	)
-	(wire
-		(pts
-			(xy 172.72 93.98) (xy 185.42 93.98)
-		)
-		(stroke
-			(width 0)
-			(type default)
-		)
-	)
-	(wire
-		(pts
-			(xy 86.36 93.98) (xy 99.06 93.98)
-		)
-		(stroke
-			(width 0)
-			(type default)
-		)
-	)
-	(wire
-		(pts
-			(xy 144.78 93.98) (xy 157.48 93.98)
-		)
-		(stroke
-			(width 0)
-			(type default)
-		)
-	)
-	(wire
-		(pts
-			(xy 198.12 93.98) (xy 210.82 93.98)
-		)
-		(stroke
-			(width 0)
-			(type default)
-		)
-	)
-	(wire
-		(pts
-			(xy 114.3 109.22) (xy 111.76 109.22)
-		)
-		(stroke
-			(width 0)
-			(type default)
-		)
-	)
-	(wire
-		(pts
-			(xy 198.12 93.98) (xy 198.12 96.52)
-		)
-		(stroke
-			(width 0)
-			(type default)
-		)
-	)
-	(wire
-		(pts
-			(xy 144.78 104.14) (xy 172.72 104.14)
-		)
-		(stroke
-			(width 0)
-			(type default)
-		)
-	)
-	(wire
-		(pts
-			(xy 73.66 101.6) (xy 73.66 104.14)
-		)
-		(stroke
-			(width 0)
-			(type default)
-		)
-	)
-	(wire
-		(pts
-			(xy 172.72 106.68) (xy 172.72 109.22)
-		)
-		(stroke
-			(width 0)
-			(type default)
-		)
-	)
-	(wire
-		(pts
-			(xy 73.66 93.98) (xy 73.66 96.52)
 		)
 		(stroke
@@
 	(hierarchical_label "VIN"
 		(shape input)
-		(at 71.12 93.98 180)
+		(at 83.82 93.98 180)
 		(effects
 			(font
@@
 	(symbol
 		(lib_id "Device:C_Small")
-		(at 73.66 99.06 0)
-		(unit 1)
-		(exclude_from_sim no)
-		(in_bom yes)
-		(on_board yes)
-		(dnp no)
-		(property "Reference" "C1201"
-			(at 76.2 97.7962 0)
-			(effects
-				(font
-					(size 1.27 1.27)
-				)
-				(justify left)
-			)
-		)
-		(property "Value" "4u7"
-			(at 76.2 100.3362 0)
-			(effects
-				(font
-					(size 1.27 1.27)
-				)
-				(justify left)
-			)
-		)
-		(property "Footprint" "Capacitor_SMD:C_0402_1005Metric"
-			(at 73.66 99.06 0)
-			(effects
-				(font
-					(size 1.27 1.27)
-				)
-				(hide yes)
-			)
-		)
-		(property "Datasheet" "~"
-			(at 73.66 99.06 0)
-			(effects
-				(font
-					(size 1.27 1.27)
-				)
-				(hide yes)
-			)
-		)
-		(property "Description" "Unpolarized capacitor, small symbol"
-			(at 73.66 99.06 0)
-			(effects
-				(font
-					(size 1.27 1.27)
-				)
-				(hide yes)
-			)
-		)
-		(pin "1"
-		)
-		(pin "2"
-		)
-		(instances
-			(project "switch_main_v5"
-				(path "/a5e57332-4284-4d3c-ab3c-13bc0ddb29b6/b1ff42f5-7cae-489e-9f8e-588cc93f3151/d017dddd-15df-4565-b589-89c8c78bc85c/2252118a-c5a3-408c-aeca-1ee5151f8202"
-					(reference "C1201")
-					(unit 1)
-				)
-				(path "/a5e57332-4284-4d3c-ab3c-13bc0ddb29b6/b1ff42f5-7cae-489e-9f8e-588cc93f3151/d017dddd-15df-4565-b589-89c8c78bc85c/b17ca951-65d8-4c7f-84f6-57bb88a8a712"
-					(reference "C3001")
-					(unit 1)
-				)
-			)
-		)
-	)
-	(symbol
-		(lib_id "Device:C_Small")
 		(at 185.42 99.06 0)
 		(unit 1)
@@
 	(symbol
 		(lib_id "power:GND1")
-		(at 73.66 106.68 0)
+		(at 86.36 106.68 0)
 		(mirror y)
 		(unit 1)
@@
 		(fields_autoplaced yes)
 		(property "Reference" "#PWR01201"
-			(at 73.66 113.03 0)
+			(at 86.36 113.03 0)
 			(effects
 				(font
@@
 		)
 		(property "Value" "GND1"
-			(at 73.66 111.76 0)
+			(at 86.36 111.76 0)
 			(effects
 				(font
@@
 		)
 		(property "Footprint" ""
-			(at 73.66 106.68 0)
+			(at 86.36 106.68 0)
 			(effects
 				(font
@@
 		)
 		(property "Datasheet" ""
-			(at 73.66 106.68 0)
+			(at 86.36 106.68 0)
 			(effects
 				(font
@@
 		)
 		(property "Description" "Power symbol creates a global label with name \"GND1\" , ground"
-			(at 73.66 106.68 0)
-			(effects
-				(font
+			(at 86.36 106.68 0)
+			(effects
+				(font

Commit message: 1V0 Rail done
Parts:
- removed C1203: 4u7, Capacitor_SMD:C_0402_1005Metric, symbol Device:C_Small
- added C1201: 4u7, Capacitor_SMD:C_0402_1005Metric, symbol Device:C_Small
Connections:
- net GND1: now also C1201.2
- net VIN: now also C1201.1
- net FB_1V8 renamed FB
- net SW_1V8 renamed SW
Other:
- moved on the sheet: C1202

Commit message: Placed most remaining passives and test points
Connections:
- net GND1: no longer U1201.2 (MODE)
- net VIN: now also U1201.2 (MODE)
Changed lines of the file:
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@@
+	)
+	(junction
+		(at 111.76 104.14)
+		(diameter 0)
+		(color 0 0 0 0)
 	)
 	(junction
@@
 	)
 	(junction
-		(at 111.76 114.3)
-		(diameter 0)
-		(color 0 0 0 0)
-	)
-	(junction
 		(at 172.72 106.68)
 		(diameter 0)
@@
 	(wire
 		(pts
-			(xy 111.76 109.22) (xy 111.76 114.3)
-		)
-		(stroke
-			(width 0)
-			(type default)
-		)
-	)
-	(wire
-		(pts
 			(xy 111.76 114.3) (xy 111.76 116.84)
 		)
@@
 		)
 		(stroke
+			(width 0)
+			(type default)
+		)
+	)
+	(wire
+		(pts
+			(xy 111.76 104.14) (xy 111.76 109.22)
+		)
+		(stroke

Commit message: Tidied schematic and PCB
Parts:
- renumbered C1201 to C601, C1202 to C602, C1204 to C603, C1205 to C604, C1206 to C605, C1207 to C606, L1201 to L601, R1201 to R601, R1202 to R602, TP1201 to TP601, U1201 to U601
