File: switch_main_v5/isolation-crossing.kicad_sch (KiCad schematic)
At the start: 6 parts, among them U2501 ISO6521REUR, U2502 ISO6520REUR

Commit message: Tidied schematic and PCB
Parts:
- renumbered C2501 to C3701, C2503 to C3702, C2502 to C3703, C2504 to C3704, U2501 to U3701, U2502 to U3702
Changed lines of the file:
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@@
 		(dnp no)
 		(fields_autoplaced yes)
-		(property "Reference" "#PWR02508"
+		(property "Reference" "#PWR03712"
 			(at 157.48 133.35 0)
 			(effects
@@
 			(project "switch_main_v4"
 				(path "/a5e57332-4284-4d3c-ab3c-13bc0ddb29b6/dfc8dd40-a5e5-401a-a1d8-3203b89e0aa2"
-					(reference "#PWR02508")
+					(reference "#PWR03712")
 					(unit 1)
 				)
@@
 		(dnp no)
 		(fields_autoplaced yes)
-		(property "Reference" "#PWR02502"
+		(property "Reference" "#PWR03703"
 			(at 101.6 97.79 0)
 			(effects
@@
 			(project "switch_main_v4"
 				(path "/a5e57332-4284-4d3c-ab3c-13bc0ddb29b6/dfc8dd40-a5e5-401a-a1d8-3203b89e0aa2"
-					(reference "#PWR02502")
+					(reference "#PWR03703")
 					(unit 1)
 				)
@@
 		(dnp no)
 		(fields_autoplaced yes)
-		(property "Reference" "#PWR02504"
+		(property "Reference" "#PWR03709"
 			(at 101.6 128.27 0)
 			(effects
@@
 			(project "switch_main_v4"
 				(path "/a5e57332-4284-4d3c-ab3c-13bc0ddb29b6/dfc8dd40-a5e5-401a-a1d8-3203b89e0aa2"
-					(reference "#PWR02504")
+					(reference "#PWR03709")
 					(unit 1)
 				)
@@
 		(dnp no)
 		(fields_autoplaced yes)
-		(property "Reference" "#PWR02511"
+		(property "Reference" "#PWR03708"
 			(at 182.88 113.03 0)
 			(effects
@@
 			(project "switch_main_v4"
 				(path "/a5e57332-4284-4d3c-ab3c-13bc0ddb29b6/dfc8dd40-a5e5-401a-a1d8-3203b89e0aa2"
-					(reference "#PWR02511")
+					(reference "#PWR03708")
 					(unit 1)
 				)
@@
 		(dnp no)
 		(fields_autoplaced yes)
-		(property "Reference" "#PWR02509"
+		(property "Reference" "#PWR03702"
 			(at 182.88 82.55 0)
 			(effects
@@
 			(project ""
 				(path "/a5e57332-4284-4d3c-ab3c-13bc0ddb29b6/dfc8dd40-a5e5-401a-a1d8-3203b89e0aa2"
-					(reference "#PWR02509")
+					(reference "#PWR03702")
 					(unit 1)
 				)
@@
 		(dnp no)
 		(fields_autoplaced yes)
-		(property "Reference" "#PWR02503"
+		(property "Reference" "#PWR03707"
 			(at 101.6 113.03 0)
 			(effects
@@
 			(project "switch_main_v4"
 				(path "/a5e57332-4284-4d3c-ab3c-13bc0ddb29b6/dfc8dd40-a5e5-401a-a1d8-3203b89e0aa2"
-					(reference "#PWR02503")
+					(reference "#PWR03707")
 					(unit 1)
 				)
@@
 		(dnp no)
 		(fields_autoplaced yes)
-		(property "Reference" "#PWR02510"
+		(property "Reference" "#PWR03704"
 			(at 182.88 97.79 0)
 			(effects
@@
 			(project "switch_main_v4"
 				(path "/a5e57332-4284-4d3c-ab3c-13bc0ddb29b6/dfc8dd40-a5e5-401a-a1d8-3203b89e0aa2"
-					(reference "#PWR02510")
+					(reference "#PWR03704")
 					(unit 1)
 				)
@@
 		(dnp no)
 		(fields_autoplaced yes)
-		(property "Reference" "U2501"
+		(property "Reference" "U3701"
 			(at 142.24 73.66 0)
 			(effects
@@
 			(project "switch_main_v4"
 				(path "/a5e57332-4284-4d3c-ab3c-13bc0ddb29b6/dfc8dd40-a5e5-401a-a1d8-3203b89e0aa2"
-					(reference "U2501")
+					(reference "U3701")
 					(unit 1)
 				)
@@
 		(dnp no)
 		(fields_autoplaced yes)
-		(property "Reference" "#PWR02501"
+		(property "Reference" "#PWR03701"
 			(at 101.6 82.55 0)
 			(effects
@@
 			(project ""
 				(path "/a5e57332-4284-4d3c-ab3c-13bc0ddb29b6/dfc8dd40-a5e5-401a-a1d8-3203b89e0aa2"
-					(reference "#PWR02501")
+					(reference "#PWR03701")
 					(unit 1)
 				)
@@
 		(dnp no)
 		(fields_autoplaced yes)
-		(property "Reference" "C2501"
+		(property "Reference" "C3701"
 			(at 104.14 85.0962 0)
 			(effects
@@
 			(project "switch_main_v4"
 				(path "/a5e57332-4284-4d3c-ab3c-13bc0ddb29b6/dfc8dd40-a5e5-401a-a1d8-3203b89e0aa2"
-					(reference "C2501")
+					(reference "C3701")
 					(unit 1)
 				)
@@
 		(dnp no)
 		(fields_autoplaced yes)
-		(property "Reference" "C2503"
+		(property "Reference" "C3702"
 			(at 185.42 85.0962 0)
 			(effects
@@
 			(project "switch_main_v4"
 				(path "/a5e57332-4284-4d3c-ab3c-13bc0ddb29b6/dfc8dd40-a5e5-401a-a1d8-3203b89e0aa2"
-					(reference "C2503")
+					(reference "C3702")
 					(unit 1)
 				)
@@
 		(dnp no)
 		(fields_autoplaced yes)
-		(property "Reference" "#PWR02505"
+		(property "Reference" "#PWR03705"
 			(at 127 102.87 0)
 			(effects
@@
 			(project "switch_main_v4"
 				(path "/a5e57332-4284-4d3c-ab3c-13bc0ddb29b6/dfc8dd40-a5e5-401a-a1d8-3203b89e0aa2"
-					(reference "#PWR02505")
+					(reference "#PWR03705")
 					(unit 1)
 				)
@@
 		(dnp no)
 		(fields_autoplaced yes)
-		(property "Reference" "C2504"
+		(property "Reference" "C3704"
 			(at 185.42 115.5762 0)
 			(effects
@@
 			(project "switch_main_v4"
 				(path "/a5e57332-4284-4d3c-ab3c-13bc0ddb29b6/dfc8dd40-a5e5-401a-a1d8-3203b89e0aa2"
-					(reference "C2504")
+					(reference "C3704")
 					(unit 1)
 				)
@@
 		(dnp no)
 		(fields_autoplaced yes)
-		(property "Reference" "#PWR02507"
+		(property "Reference" "#PWR03706"
 			(at 157.48 102.87 0)
 			(effects
@@
 			(project ""
 				(path "/a5e57332-4284-4d3c-ab3c-13bc0ddb29b6/dfc8dd40-a5e5-401a-a1d8-3203b89e0aa2"
-					(reference "#PWR02507")
+					(reference "#PWR03706")
 					(unit 1)
 				)
@@
 		(dnp no)
 		(fields_autoplaced yes)
-		(property "Reference" "#PWR02512"
+		(property "Reference" "#PWR03710"
 			(at 182.88 128.27 0)
 			(effects
@@
 			(project "switch_main_v4"
 				(path "/a5e57332-4284-4d3c-ab3c-13bc0ddb29b6/dfc8dd40-a5e5-401a-a1d8-3203b89e0aa2"
-					(reference "#PWR02512")
+					(reference "#PWR03710")
 					(unit 1)
 				)
@@
 		(dnp no)
 		(fields_autoplaced yes)
-		(property "Reference" "#PWR02506"
+		(property "Reference" "#PWR03711"
 			(at 127 133.35 0)
 			(effects
@@
 			(project "switch_main_v4"
 				(path "/a5e57332-4284-4d3c-ab3c-13bc0ddb29b6/dfc8dd40-a5e5-401a-a1d8-3203b89e0aa2"
-					(reference "#PWR02506")
+					(reference "#PWR03711")
 					(unit 1)
 				)
@@
 		(dnp no)
 		(fields_autoplaced yes)
-		(property "Reference" "C2502"
+		(property "Reference" "C3703"
 			(at 104.14 115.5762 0)
 			(effects
@@
 			(project "switch_main_v4"
 				(path "/a5e57332-4284-4d3c-ab3c-13bc0ddb29b6/dfc8dd40-a5e5-401a-a1d8-3203b89e0aa2"
-					(reference "C2502")
+					(reference "C3703")
 					(unit 1)
 				)
@@
 		(dnp no)
 		(fields_autoplaced yes)
-		(property "Reference" "U2502"
+		(property "Reference" "U3702"
 			(at 142.24 104.14 0)
 			(effects
@@
 			(project ""
 				(path "/a5e57332-4284-4d3c-ab3c-13bc0ddb29b6/dfc8dd40-a5e5-401a-a1d8-3203b89e0aa2"
-					(reference "U2502")
-					(unit 1)
-				)
+					(reference "U3702")
+					(unit 1)
+				)
