File: switch_main_v5/mpoe-1-channel.kicad_sch (KiCad schematic)
At the start: 18 parts, among them Q2301 DMN21D2UFB-7B, Q2302 DMP21D0UFB-7B, U2301 NCS213RMUTAG, U2302 TPS27S100BRRK

Commit message: Tidied schematic and PCB
Parts:
- renumbered C2302 to C3101, C2301 to C3102, D2301 to D3101, F2301 to F3101, Q2302 to Q3101, Q2301 to Q3102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
