File: switch_main_v5/podl-2-channels.kicad_sch (KiCad schematic)
At the start: 37 parts, among them Q2201 DMP21D0UFB-7B, Q2202 DMP21D0UFB-7B, Q2203 DMN21D2UFB-7B, Q2204 DMP21D0UFB-7B, Q2205 DMN21D2UFB-7B, Q2206 DMP21D0UFB-7B, U2201 TPS27S100BRRK, U2202 TPS27S100BRRK

Commit message: MDIO multiplexing
Parts:
- renumbered C2201 to C, C2202 to C, D2201 to D, D2202 to D, Q2201 to Q, Q2205 to Q, Q2206 to Q, Q2202 to Q, Q2203 to Q, Q2204 to Q, R2203 to R, R2219 to R, R2209 to R, R2223 to R, R2221 to R, R2201 to R, R2215 to R, R2204 to R, R2222 to R, R2202 to R, R2214 to R, R2206 to R, R2212 to R, R2216 to R, R2218 to R, R2220 to R, R2205 to R, R2210 to R, R2217 to R, R2213 to R, R2211 to R, R2207 to R, R2208 to R, U2202 to U, U2201 to U, Z2201 to Z, Z2202 to Z

Commit message: Started updating regulators for v5
Parts:
- renumbered C to C?, D to D?, Q to Q?, R to R?, U to U?, Z to Z?

Commit message: Updated 1v0_buck_converter feedback resistors
Parts:
- gave numbers to parts that had none: 37

Commit message: Tidied schematic and PCB
Parts:
- renumbered C2201 to C3001, C2202 to C3002, D2201 to D3001, D2202 to D3002, Q2201 to Q3001, Q2202 to Q3002, Q2204 to Q3003, Q2206 to Q3004, Q2203 to Q3005, Q2205 to Q3006, R2205 to R3001, R2209 to R3002, R2220 to R3003, R2208 to R3004, R2219 to R3005, R2207 to R3006, R2218 to R3007, R2202 to R3008, R2211 to R3009, R2214 to R3010, R2222 to R3011, R2203 to R3012, R2210 to R3013, R2215 to R3014, R2221 to R3015, R2204 to R3016, R2212 to R3017, R2216 to R3018, R2223 to R3019, R2201 to R3020, R2206 to R3021, R2213 to R3022, R2217 to R3023, U2201 to U3001, U2202 to U3002, Z2201 to Z3001, Z2202 to Z3002
