File: switch_main_v5/power-3v3-regulators.kicad_sch (KiCad schematic)
At the start: 25 parts, among them U401 TPS7B8133QDRVRQ1, U402 LMQ66420MC3RXBRQ1, U403 TPS2116DRL

Commit message: Started updating regulators for v5
Changed lines of the file:
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@@
+		)
+	)
+	(text_box "Change to 3A"
+		(exclude_from_sim no)
+		(at 149.86 33.02 0)
+		(size 10.16 5.08)
+		(margins 0.9525 0.9525 0.9525 0.9525)
+		(stroke
+			(width 0)
+			(type solid)
+			(color 255 0 0 1)
+		)
+		(fill
+			(type none)
+		)
+		(effects
+			(font
+				(size 1.27 1.27)
+				(color 255 0 0 1)
+			)
 		)
 	)

Commit message: Updated 1v0_buck_converter feedback resistors
Parts:
- renumbered C404 to C403, C403 to C404, TP806 to TP403, U402 to U401, U401 to U402
Changed lines of the file:
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@@
 		(on_board yes)
 		(dnp no)
-		(property "Reference" "C404"
+		(property "Reference" "C403"
 			(at 81.28 72.3962 0)
 			(effects
@@
 			(project "switch_main_v4"
 				(path "/a5e57332-4284-4d3c-ab3c-13bc0ddb29b6/b1ff42f5-7cae-489e-9f8e-588cc93f3151/3215d643-ce31-476b-aa01-9096c7ce3dfb"
-					(reference "C404")
+					(reference "C403")
 					(unit 1)
 				)
@@
 		(dnp no)
 		(fields_autoplaced yes)
-		(property "Reference" "#PWR0410"
+		(property "Reference" "#PWR0408"
 			(at 127 87.63 0)
 			(effects
@@
 			(project "switch_main_v4"
 				(path "/a5e57332-4284-4d3c-ab3c-13bc0ddb29b6/b1ff42f5-7cae-489e-9f8e-588cc93f3151/3215d643-ce31-476b-aa01-9096c7ce3dfb"
-					(reference "#PWR0410")
+					(reference "#PWR0408")
 					(unit 1)
 				)
@@
 		(on_board yes)
 		(dnp no)
-		(property "Reference" "C403"
+		(property "Reference" "C404"
 			(at 83.82 134.62 0)
 			(effects
@@
 			(project "switch_main_v4"
 				(path "/a5e57332-4284-4d3c-ab3c-13bc0ddb29b6/b1ff42f5-7cae-489e-9f8e-588cc93f3151/3215d643-ce31-476b-aa01-9096c7ce3dfb"
-					(reference "C403")
+					(reference "C404")
 					(unit 1)
 				)
@@
 		(on_board yes)
 		(dnp no)
-		(property "Reference" "TP806"
+		(property "Reference" "TP403"
 			(at 269.24 50.8 0)
 			(effects
@@
 			(project "switch_main_v4"
 				(path "/a5e57332-4284-4d3c-ab3c-13bc0ddb29b6/b1ff42f5-7cae-489e-9f8e-588cc93f3151/3215d643-ce31-476b-aa01-9096c7ce3dfb"
-					(reference "TP806")
+					(reference "TP403")
 					(unit 1)
 				)
@@
 		(dnp no)
 		(fields_autoplaced yes)
-		(property "Reference" "U402"
+		(property "Reference" "U401"
 			(at 104.14 35.56 0)
 			(effects
@@
 			(project ""
 				(path "/a5e57332-4284-4d3c-ab3c-13bc0ddb29b6/b1ff42f5-7cae-489e-9f8e-588cc93f3151/3215d643-ce31-476b-aa01-9096c7ce3dfb"
-					(reference "U402")
+					(reference "U401")
 					(unit 1)
 				)
@@
 		(dnp no)
 		(fields_autoplaced yes)
-		(property "Reference" "#PWR0406"
+		(property "Reference" "#PWR0404"
 			(at 78.74 87.63 0)
 			(effects
@@
 			(project "switch_main_v4"
 				(path "/a5e57332-4284-4d3c-ab3c-13bc0ddb29b6/b1ff42f5-7cae-489e-9f8e-588cc93f3151/3215d643-ce31-476b-aa01-9096c7ce3dfb"
-					(reference "#PWR0406")
+					(reference "#PWR0404")
 					(unit 1)
 				)
@@
 		(dnp no)
 		(fields_autoplaced yes)
-		(property "Reference" "#PWR0405"
+		(property "Reference" "#PWR0406"
 			(at 81.28 148.59 0)
 			(effects
@@
 			(project "switch_main_v4"
 				(path "/a5e57332-4284-4d3c-ab3c-13bc0ddb29b6/b1ff42f5-7cae-489e-9f8e-588cc93f3151/3215d643-ce31-476b-aa01-9096c7ce3dfb"
-					(reference "#PWR0405")
+					(reference "#PWR0406")
 					(unit 1)
 				)
@@
 		(dnp no)
 		(fields_autoplaced yes)
-		(property "Reference" "#PWR0408"
+		(property "Reference" "#PWR0409"
 			(at 127 161.29 0)
 			(effects
@@
 			(project "switch_main_v4"
 				(path "/a5e57332-4284-4d3c-ab3c-13bc0ddb29b6/b1ff42f5-7cae-489e-9f8e-588cc93f3151/3215d643-ce31-476b-aa01-9096c7ce3dfb"
-					(reference "#PWR0408")
+					(reference "#PWR0409")
 					(unit 1)
 				)
@@
 		(dnp no)
 		(fields_autoplaced yes)
-		(property "Reference" "U401"
+		(property "Reference" "U402"
 			(at 109.22 124.46 0)
 			(effects
@@
 			(project "switch_main_v4"
 				(path "/a5e57332-4284-4d3c-ab3c-13bc0ddb29b6/b1ff42f5-7cae-489e-9f8e-588cc93f3151/3215d643-ce31-476b-aa01-9096c7ce3dfb"
-					(reference "U401")
+					(reference "U402")
 					(unit 1)
 				)
@@
 		(dnp no)
 		(fields_autoplaced yes)
-		(property "Reference" "#PWR0404"
+		(property "Reference" "#PWR0405"
 			(at 81.28 133.35 0)
 			(effects
@@
 			(project "switch_main_v4"
 				(path "/a5e57332-4284-4d3c-ab3c-13bc0ddb29b6/b1ff42f5-7cae-489e-9f8e-588cc93f3151/3215d643-ce31-476b-aa01-9096c7ce3dfb"
-					(reference "#PWR0404")
+					(reference "#PWR0405")
 					(unit 1)
 				)
@@
 		(dnp no)
 		(fields_autoplaced yes)
-		(property "Reference" "#PWR0409"
+		(property "Reference" "#PWR0410"
 			(at 132.08 148.59 0)
 			(effects
@@
 			(project "switch_main_v4"
 				(path "/a5e57332-4284-4d3c-ab3c-13bc0ddb29b6/b1ff42f5-7cae-489e-9f8e-588cc93f3151/3215d643-ce31-476b-aa01-9096c7ce3dfb"
-					(reference "#PWR0409")
-					(unit 1)
-				)
+					(reference "#PWR0410")
+					(unit 1)
+				)

Commit message: Changed main 3V3 regulator to 3A, added switch 2 crystal & other changes
Parts:
- removed L401: 74438323022, project_footprints:L_Wurth_WE-MAPI-2510, symbol PWR-IND:2510_74438323022
- removed U401: LMQ66420MC3RXBRQ1, project_footprints:LMQ664x0, symbol PWR-SMPS:LMQ66420MC3RXBRQ1
- added L401: 74479335329222, project_footprints:L_Wurth_WE-PMFI-353220, symbol PWR-IND:353220_74479335329222
- added U401: LMQ66430MC3RXBRQ1, project_footprints:LMQ664x0, symbol PWR-SMPS:LMQ66430MC3RXBRQ1
Connections:
- net +3V3: now also L401.2, U401.11 (VOUT/FB)
- net +VIN: now also U401.3 (VIN)
- net 3V3_PG: now also U401.14 (PG)
- net EN: now also U401.1 (EN/UVLO), U401.16 (EN/UVLO)
- net GND1: now also U401.15 (GND/DAP), U401.6 (PGND)
- net MODE: now also U401.13 (MODE/SYNC)
- net SW: now also L401.1, U401.7 (SW)
- net VCC: now also U401.10 (VCC)
- new net: U401.18 (BOOT), U401.8 (BOOT)

Commit message: Tidied schematic and PCB
Parts:
- renumbered C406 to C403, C407 to C404, C408 to C405, C409 to C406, C410 to C407, C411 to C408, C412 to C409, C413 to C410, C414 to C411, C415 to C412, C403 to C413, C404 to C414, C405 to C415, TP402 to TP401, TP403 to TP402, TP401 to TP403, U403 to U402, U402 to U403
Other:
- moved on the sheet: C401, C402, C403, C404, C405, C406, C407, C408, C409, C410, C411, C412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
