File: switch_main_v5/power-in.kicad_sch (KiCad schematic)
At the start: 13 parts, among them J301 MKXS1-1 Power Input, U301 TVS3301DRBR, U302 TPS26600RHFR

Commit message: Updated 1v0_buck_converter feedback resistors
Parts:
- renumbered R309 to R308
Changed lines of the file:
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@@
 		(on_board yes)
 		(dnp no)
-		(property "Reference" "R309"
+		(property "Reference" "R308"
 			(at 254 85.09 0)
 			(effects
@@
 			(project "switch_main_v4"
 				(path "/a5e57332-4284-4d3c-ab3c-13bc0ddb29b6/b1ff42f5-7cae-489e-9f8e-588cc93f3151/7660ee4b-63c9-4370-ad91-90cac1411452"
-					(reference "R309")
+					(reference "R308")
 					(unit 1)
 				)
@@
 		(dnp no)
 		(fields_autoplaced yes)
-		(property "Reference" "#PWR0306"
+		(property "Reference" "#PWR0305"
 			(at 251.46 97.79 0)
 			(effects
@@
 			(project "switch_main_v4"
 				(path "/a5e57332-4284-4d3c-ab3c-13bc0ddb29b6/b1ff42f5-7cae-489e-9f8e-588cc93f3151/7660ee4b-63c9-4370-ad91-90cac1411452"
-					(reference "#PWR0306")
+					(reference "#PWR0305")
 					(unit 1)
 				)
@@
 		(dnp no)
 		(fields_autoplaced yes)
-		(property "Reference" "#PWR0307"
+		(property "Reference" "#PWR0304"
 			(at 251.46 72.39 0)
 			(effects
@@
 			(project "switch_main_v4"
 				(path "/a5e57332-4284-4d3c-ab3c-13bc0ddb29b6/b1ff42f5-7cae-489e-9f8e-588cc93f3151/7660ee4b-63c9-4370-ad91-90cac1411452"
-					(reference "#PWR0307")
+					(reference "#PWR0304")
 					(unit 1)
 				)
@@
 		(dnp no)
 		(fields_autoplaced yes)
-		(property "Reference" "#PWR0304"
+		(property "Reference" "#PWR0303"
 			(at 210.82 118.11 0)
 			(effects
@@
 			(project "switch_main_v4"
 				(path "/a5e57332-4284-4d3c-ab3c-13bc0ddb29b6/b1ff42f5-7cae-489e-9f8e-588cc93f3151/7660ee4b-63c9-4370-ad91-90cac1411452"
-					(reference "#PWR0304")
-					(unit 1)
-				)
+					(reference "#PWR0303")
+					(unit 1)
+				)

Commit message: Changed main 3V3 regulator to 3A, added switch 2 crystal & other changes
Changed lines of the file:
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@@
 	(symbol
 		(lib_id "TVS:SZESD7241N2T5G")
-		(at 71.12 81.28 90)
+		(at 73.66 81.28 90)
 		(unit 1)
 		(exclude_from_sim no)
@@
 		(on_board yes)
 		(dnp no)
-		(fields_autoplaced yes)
 		(property "Reference" "D301"
-			(at 76.2 80.0099 90)
+			(at 76.2 80.01 90)
 			(effects
 				(font
@@
 		)
 		(property "Value" "SZESD7241N2T5G"
-			(at 76.2 82.5499 90)
+			(at 76.2 82.55 90)
 			(effects
 				(font
@@
 		)
 		(property "Footprint" "project_footprints:SZESD7462N2T5G"
-			(at 81.28 97.79 0)
+			(at 83.82 97.79 0)
 			(effects
 				(font
@@
 		)
 		(property "Datasheet" "https://www.onsemi.com/pub/Collateral/ESD7241-D.PDF"
-			(at 83.82 110.49 0)
+			(at 86.36 110.49 0)
 			(effects
 				(font
@@
 		)
 		(property "Description" "SZESD7241MXWT5G Wettable Flank Package; SZ Prefix for Automotive and Other Applications Requiring Unique Site and Control Change Requirements; AECQ101 Qualified and PPAP CapableSZ Prefix for Automotive and Other Applications Requiring Unique Site and Control Change Requirements; AECQ101 Qualified and PPAP Capable; Ultra-Low Capacitance: < 1.0pF Max; Low Leakage: < 0.5uA; IEC61000-4-2 (ESD): Level 4 +/-28kV Contact; IEC61000-4-4 (EFT): 40A - 5/50ns; IEC61000-4-5 (Lightning): 1A - 8/20us; These Devices are Pb"
-			(at 77.47 81.28 0)
+			(at 80.01 81.28 0)
 			(effects
 				(font
@@
 		)
 		(property "Height" "0.4"
-			(at 86.36 82.55 0)
+			(at 88.9 82.55 0)
 			(effects
 				(font
@@
 		)
 		(property "Mouser Part Number" "863-SZESD7241N2T5G"
-			(at 88.9 92.71 0)
+			(at 91.44 92.71 0)
 			(effects
 				(font
@@
 		)
 		(property "Mouser Price/Stock" "https://www.mouser.co.uk/ProductDetail/onsemi/SZESD7241N2T5G?qs=z6PAvqrnkvSq0oMCl81g4Q%3D%3D"
-			(at 91.44 130.81 0)
+			(at 93.98 130.81 0)
 			(effects
 				(font
@@
 		)
 		(property "Manufacturer_Name" "onsemi"
-			(at 93.98 85.09 0)
+			(at 96.52 85.09 0)
 			(effects
 				(font
@@
 		)
 		(property "Manufacturer_Part_Number" "SZESD7241N2T5G"
-			(at 96.52 90.17 0)
+			(at 99.06 90.17 0)
 			(effects
 				(font

Commit message: Placed 1000BASE-T PHY decoupling capacitors
Parts:
- J301: footprint project_footprints:10132798-031100LF -> project_footprints:10132797-031100LF
Changed lines of the file:
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@@
 			)
 		)
-		(property "Footprint" "project_footprints:10132798-031100LF"
+		(property "Footprint" "project_footprints:10132797-031100LF"
 			(at 43.18 88.9 0)
 			(effects

Commit message: Changed primary side input current limit to 545mA (from 255mA which is less than the max possible load current of 326mA)
Parts:
- R304: value 47k -> 22k
Changed lines of the file:
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@@
 		)
 	)
-	(text_box "R_{ILIM} = 47kΩ ∴ I_{LIM} = 285mA"
+	(text_box "R_{ILIM} = 22kΩ\n∴ I_{LIM} = 12 / 22 = 545mA"
 		(exclude_from_sim no)
 		(at 238.76 111.76 0)
-		(size 17.78 5.08)
+		(size 30.48 5.08)
 		(margins 0.9525 0.9525 0.9525 0.9525)
 		(stroke
@@
 			)
 		)
-		(property "Value" "47k"
+		(property "Value" "22k"
 			(at 218.44 107.9501 0)
 			(effects

Commit message: Tidied schematic and PCB
Parts:
- renumbered R307 to R301, R301 to R302, R308 to R303, R302 to R304, R306 to R305, R303 to R306, R304 to R307, R305 to R308, U302 to U301, U301 to U302
Changed lines of the file:
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@@
 		(dnp no)
 		(fields_autoplaced yes)
-		(property "Reference" "#PWR0301"
+		(property "Reference" "#PWR0304"
 			(at 109.22 100.33 0)
 			(effects
@@
 			(project "switch_main_v4"
 				(path "/a5e57332-4284-4d3c-ab3c-13bc0ddb29b6/b1ff42f5-7cae-489e-9f8e-588cc93f3151/7660ee4b-63c9-4370-ad91-90cac1411452"
-					(reference "#PWR0301")
+					(reference "#PWR0304")
 					(unit 1)
 				)
@@
 		(on_board yes)
 		(dnp no)
-		(property "Reference" "R308"
+		(property "Reference" "R303"
 			(at 254 85.09 0)
 			(effects
@@
 			(project "switch_main_v4"
 				(path "/a5e57332-4284-4d3c-ab3c-13bc0ddb29b6/b1ff42f5-7cae-489e-9f8e-588cc93f3151/7660ee4b-63c9-4370-ad91-90cac1411452"
-					(reference "R308")
+					(reference "R303")
 					(unit 1)
 				)
@@
 		(on_board yes)
 		(dnp no)
-		(property "Reference" "R303"
+		(property "Reference" "R306"
 			(at 167.64 97.7899 0)
 			(effects
@@
 			(project "switch_main_v4"
 				(path "/a5e57332-4284-4d3c-ab3c-13bc0ddb29b6/b1ff42f5-7cae-489e-9f8e-588cc93f3151/7660ee4b-63c9-4370-ad91-90cac1411452"
-					(reference "R303")
+					(reference "R306")
 					(unit 1)
 				)
@@
 		(dnp no)
 		(fields_autoplaced yes)
-		(property "Reference" "#PWR0305"
+		(property "Reference" "#PWR0303"
 			(at 251.46 97.79 0)
 			(effects
@@
 			(project "switch_main_v4"
 				(path "/a5e57332-4284-4d3c-ab3c-13bc0ddb29b6/b1ff42f5-7cae-489e-9f8e-588cc93f3151/7660ee4b-63c9-4370-ad91-90cac1411452"
-					(reference "#PWR0305")
+					(reference "#PWR0303")
 					(unit 1)
 				)
@@
 		(on_board yes)
 		(dnp no)
-		(property "Reference" "R304"
+		(property "Reference" "R307"
 			(at 218.44 105.4101 0)
 			(effects
@@
 			(project "switch_main_v4"
 				(path "/a5e57332-4284-4d3c-ab3c-13bc0ddb29b6/b1ff42f5-7cae-489e-9f8e-588cc93f3151/7660ee4b-63c9-4370-ad91-90cac1411452"
-					(reference "R304")
+					(reference "R307")
 					(unit 1)
 				)
@@
 		(on_board yes)
 		(dnp no)
-		(property "Reference" "R302"
+		(property "Reference" "R304"
 			(at 167.64 87.6299 0)
 			(effects
@@
 			(project "switch_main_v4"
 				(path "/a5e57332-4284-4d3c-ab3c-13bc0ddb29b6/b1ff42f5-7cae-489e-9f8e-588cc93f3151/7660ee4b-63c9-4370-ad91-90cac1411452"
-					(reference "R302")
+					(reference "R304")
 					(unit 1)
 				)
@@
 		(dnp no)
 		(fields_autoplaced yes)
-		(property "Reference" "U301"
+		(property "Reference" "U302"
 			(at 113.03 80.0099 0)
 			(effects
@@
 			(project ""
 				(path "/a5e57332-4284-4d3c-ab3c-13bc0ddb29b6/b1ff42f5-7cae-489e-9f8e-588cc93f3151/7660ee4b-63c9-4370-ad91-90cac1411452"
-					(reference "U301")
+					(reference "U302")
 					(unit 1)
 				)
@@
 		(on_board yes)
 		(dnp no)
-		(property "Reference" "R301"
+		(property "Reference" "R302"
 			(at 167.64 77.4699 0)
 			(effects
@@
 			(project "switch_main_v4"
 				(path "/a5e57332-4284-4d3c-ab3c-13bc0ddb29b6/b1ff42f5-7cae-489e-9f8e-588cc93f3151/7660ee4b-63c9-4370-ad91-90cac1411452"
-					(reference "R301")
+					(reference "R302")
 					(unit 1)
 				)
@@
 		(dnp no)
 		(fields_autoplaced yes)
-		(property "Reference" "#PWR0304"
+		(property "Reference" "#PWR0301"
 			(at 251.46 72.39 0)
 			(effects
@@
 			(project "switch_main_v4"
 				(path "/a5e57332-4284-4d3c-ab3c-13bc0ddb29b6/b1ff42f5-7cae-489e-9f8e-588cc93f3151/7660ee4b-63c9-4370-ad91-90cac1411452"
-					(reference "#PWR0304")
+					(reference "#PWR0301")
 					(unit 1)
 				)
@@
 		(dnp no)
 		(fields_autoplaced yes)
-		(property "Reference" "#PWR0303"
+		(property "Reference" "#PWR0305"
 			(at 210.82 118.11 0)
 			(effects
@@
 			(project "switch_main_v4"
 				(path "/a5e57332-4284-4d3c-ab3c-13bc0ddb29b6/b1ff42f5-7cae-489e-9f8e-588cc93f3151/7660ee4b-63c9-4370-ad91-90cac1411452"
-					(reference "#PWR0303")
+					(reference "#PWR0305")
 					(unit 1)
 				)
@@
 		(on_board yes)
 		(dnp no)
-		(property "Reference" "R307"
+		(property "Reference" "R301"
 			(at 254 74.93 0)
 			(effects
@@
 			(project "switch_main_v4"
 				(path "/a5e57332-4284-4d3c-ab3c-13bc0ddb29b6/b1ff42f5-7cae-489e-9f8e-588cc93f3151/7660ee4b-63c9-4370-ad91-90cac1411452"
-					(reference "R307")
+					(reference "R301")
 					(unit 1)
 				)
@@
 		(on_board yes)
 		(dnp no)
-		(property "Reference" "R306"
+		(property "Reference" "R305"
 			(at 231.14 88.9 90)
 			(effects
@@
 			(project "switch_main_v4"
 				(path "/a5e57332-4284-4d3c-ab3c-13bc0ddb29b6/b1ff42f5-7cae-489e-9f8e-588cc93f3151/7660ee4b-63c9-4370-ad91-90cac1411452"
-					(reference "R306")
+					(reference "R305")
 					(unit 1)
 				)
@@
 		(dnp no)
 		(fields_autoplaced yes)
-		(property "Reference" "U302"
+		(property "Reference" "U301"
 			(at 190.5 63.5 0)
 			(effects
@@
 			(project "switch_main_v4"
 				(path "/a5e57332-4284-4d3c-ab3c-13bc0ddb29b6/b1ff42f5-7cae-489e-9f8e-588cc93f3151/7660ee4b-63c9-4370-ad91-90cac1411452"
-					(reference "U302")
+					(reference "U301")
 					(unit 1)
 				)
@@
 		(on_board yes)
 		(dnp no)
-		(property "Reference" "R305"
+		(property "Reference" "R308"
 			(at 228.6 105.4101 0)
 			(effects
@@
 			(project "switch_main_v4"
 				(path "/a5e57332-4284-4d3c-ab3c-13bc0ddb29b6/b1ff42f5-7cae-489e-9f8e-588cc93f3151/7660ee4b-63c9-4370-ad91-90cac1411452"
-					(reference "R305")
-					(unit 1)
-				)
+					(reference "R308")
+					(unit 1)
+				)
