File: switch_main_v5/power-regulators-isolated.kicad_sch (KiCad schematic)
At the start: 20 parts, among them U701 TPS7B8133QDRVRQ1, U702 MAX20075DATCA/V+, U703 NCP508MT25TBG

Commit message: Tidied schematic and PCB
Parts:
- renumbered C705 to C1301, C701 to C1302, C707 to C1303, C708 to C1304, C709 to C1305, C710 to C1306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
