File: switch_main_v5/secondary-mcu.kicad_sch (KiCad schematic)
At the start: 18 parts, among them Q2601 DMN21D2UFB-7B, Q2602 DMN21D2UFB-7B, U2601 STM32H503KBUx

Commit message: Updated 1v0_buck_converter feedback resistors
Parts:
- renumbered TP805 to TP2603, TP2603 to TP2604, TP2604 to TP2605
Changed lines of the file:
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@@
 		(on_board yes)
 		(dnp no)
-		(property "Reference" "TP2604"
+		(property "Reference" "TP2605"
 			(at 210.82 104.14 0)
 			(effects
@@
 			(project "switch_main_v4"
 				(path "/a5e57332-4284-4d3c-ab3c-13bc0ddb29b6/f1e473a5-3ec5-42ea-b224-3fef4a008a5e"
-					(reference "TP2604")
+					(reference "TP2605")
 					(unit 1)
 				)
@@
 		(on_board yes)
 		(dnp no)
-		(property "Reference" "TP805"
+		(property "Reference" "TP2603"
 			(at 106.68 101.6 0)
 			(effects
@@
 			(project "switch_main_v4"
 				(path "/a5e57332-4284-4d3c-ab3c-13bc0ddb29b6/f1e473a5-3ec5-42ea-b224-3fef4a008a5e"
-					(reference "TP805")
+					(reference "TP2603")
 					(unit 1)
 				)
@@
 		(on_board yes)
 		(dnp no)
-		(property "Reference" "TP2603"
+		(property "Reference" "TP2604"
 			(at 210.82 99.06 0)
 			(effects
@@
 			(project "switch_main_v4"
 				(path "/a5e57332-4284-4d3c-ab3c-13bc0ddb29b6/f1e473a5-3ec5-42ea-b224-3fef4a008a5e"
-					(reference "TP2603")
+					(reference "TP2604")
 					(unit 1)
 				)
@@
 		(dnp no)
 		(fields_autoplaced yes)
-		(property "Reference" "#PWR02607"
+		(property "Reference" "#PWR02608"
 			(at 205.74 67.31 0)
 			(effects
@@
 			(project ""
 				(path "/a5e57332-4284-4d3c-ab3c-13bc0ddb29b6/f1e473a5-3ec5-42ea-b224-3fef4a008a5e"
-					(reference "#PWR02607")
+					(reference "#PWR02608")
 					(unit 1)
 				)
@@
 		(dnp no)
 		(fields_autoplaced yes)
-		(property "Reference" "#PWR02611"
+		(property "Reference" "#PWR02612"
 			(at 259.08 97.79 0)
 			(effects
@@
 			(project "switch_main_v4"
 				(path "/a5e57332-4284-4d3c-ab3c-13bc0ddb29b6/f1e473a5-3ec5-42ea-b224-3fef4a008a5e"
-					(reference "#PWR02611")
+					(reference "#PWR02612")
 					(unit 1)
 				)
@@
 		(dnp no)
 		(fields_autoplaced yes)
-		(property "Reference" "#PWR02610"
+		(property "Reference" "#PWR02611"
 			(at 246.38 125.73 0)
 			(effects
@@
 			(project "switch_main_v4"
 				(path "/a5e57332-4284-4d3c-ab3c-13bc0ddb29b6/f1e473a5-3ec5-42ea-b224-3fef4a008a5e"
-					(reference "#PWR02610")
+					(reference "#PWR02611")
 					(unit 1)
 				)
@@
 		(dnp no)
 		(fields_autoplaced yes)
-		(property "Reference" "#PWR02609"
+		(property "Reference" "#PWR02610"
 			(at 233.68 107.95 0)
 			(effects
@@
 			(project "switch_main_v4"
 				(path "/a5e57332-4284-4d3c-ab3c-13bc0ddb29b6/f1e473a5-3ec5-42ea-b224-3fef4a008a5e"
-					(reference "#PWR02609")
+					(reference "#PWR02610")
 					(unit 1)
 				)
@@
 		(dnp no)
 		(fields_autoplaced yes)
-		(property "Reference" "#PWR02612"
+		(property "Reference" "#PWR02613"
 			(at 259.08 125.73 0)
 			(effects
@@
 			(project "switch_main_v4"
 				(path "/a5e57332-4284-4d3c-ab3c-13bc0ddb29b6/f1e473a5-3ec5-42ea-b224-3fef4a008a5e"
-					(reference "#PWR02612")
+					(reference "#PWR02613")
 					(unit 1)
 				)
@@
 		(dnp no)
 		(fields_autoplaced yes)
-		(property "Reference" "#PWR02613"
+		(property "Reference" "#PWR02605"
 			(at 121.92 110.49 0)
 			(effects
@@
 			(project "switch_main_v4"
 				(path "/a5e57332-4284-4d3c-ab3c-13bc0ddb29b6/f1e473a5-3ec5-42ea-b224-3fef4a008a5e"
-					(reference "#PWR02613")
+					(reference "#PWR02605")
 					(unit 1)
 				)
@@
 		(dnp no)
 		(fields_autoplaced yes)
-		(property "Reference" "#PWR02606"
+		(property "Reference" "#PWR02607"
 			(at 190.5 135.89 0)
 			(effects
@@
 			(project ""
 				(path "/a5e57332-4284-4d3c-ab3c-13bc0ddb29b6/f1e473a5-3ec5-42ea-b224-3fef4a008a5e"
-					(reference "#PWR02606")
+					(reference "#PWR02607")
 					(unit 1)
 				)
@@
 		(dnp no)
 		(fields_autoplaced yes)
-		(property "Reference" "#PWR02605"
+		(property "Reference" "#PWR02606"
 			(at 190.5 67.31 0)
 			(effects
@@
 			(project ""
 				(path "/a5e57332-4284-4d3c-ab3c-13bc0ddb29b6/f1e473a5-3ec5-42ea-b224-3fef4a008a5e"
-					(reference "#PWR02605")
+					(reference "#PWR02606")
 					(unit 1)
 				)
@@
 		(dnp no)
 		(fields_autoplaced yes)
-		(property "Reference" "#PWR02608"
+		(property "Reference" "#PWR02609"
 			(at 233.68 80.01 0)
 			(effects
@@
 			(project "switch_main_v4"
 				(path "/a5e57332-4284-4d3c-ab3c-13bc0ddb29b6/f1e473a5-3ec5-42ea-b224-3fef4a008a5e"
-					(reference "#PWR02608")
-					(unit 1)
-				)
+					(reference "#PWR02609")
+					(unit 1)
+				)

Commit message: Changed main 3V3 regulator to 3A, added switch 2 crystal & other changes
Connections:
- no-connect marks 4 -> 5
Changed lines of the file:
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@@
+	)
+	(no_connect
+		(at 142.24 111.76)
 	)
 	(no_connect

Commit message: Tidied schematic and PCB
Parts:
- renumbered C2602 to C3801, C2604 to C3802, C2606 to C3803, C2603 to C3804, C2605 to C3805, C2607 to C3806, C2601 to C3807, Q2602 to Q3801, Q2601 to Q3802, R2602 to R3801, R2603 to R3802, R2601 to R3803, TP2601 to TP3801, TP2602 to TP3802, TP2604 to TP3803, TP2603 to TP3804, TP2605 to TP3805, U2601 to U3801
