File: pcbs/switch-main-v5/switch-1.kicad_sch (KiCad schematic)
At the start: 43 parts, among them U1601 SJA1105QELY, Y1601 XRCGB25M000F3A16R0

Commit message: Fixed bug with IO voltage of connection between switch 0 and switch 1
Connections:
- net +1V8: now also C1608.1, C1609.1, C1616.1, C1617.1, C1623.1, C1624.1, U1601.G11 (VDDIO_MII3_1), U1601.H11 (VDDIO_MII3_2), U1601.K11 (VDDIO_MII3_3), U1601.L10 (VDDIO_MII4_2), U1601.L11 (VDDIO_MII4_3), U1601.L8 (VDDIO_MII4_1)
- net +3V3: no longer C1608.1, C1609.1, C1616.1, C1617.1, C1623.1, C1624.1, U1601.G11 (VDDIO_MII3_1), U1601.H11 (VDDIO_MII3_2), U1601.K11 (VDDIO_MII3_3), U1601.L10 (VDDIO_MII4_2), U1601.L11 (VDDIO_MII4_3), U1601.L8 (VDDIO_MII4_1)
