File: pcbs/switch-main-v5/switch-main-v5.kicad_pcb (KiCad board)
At the start: 6 copper layers, 93 x 50 mm, 646 parts, among them J1201 MKXS1-1 Power Input, J301 MKXS1-1 Power Input, J3601 JST-GH-2-Horizontal, J3602 JST-GH-2-Horizontal, J3603 ARJM11D7-502-AB-EW2, J3604 MSPE-J2L0-B00, J3605 MSPE-J2L0-B00, J3606 MSPE-J2L0-x00, J3607 MSPE-J2L0-x00, J3608 MSPE-J2L0-x00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

Commit message: Tidied up PCB
Routing:
- net GND1: track 117.5 -> 119.8 mm
Other:
- board text added: "26/04/2026"
- board text removed: "29/12/2025"
